File: hardware/battery_pack.kicad_sch (KiCad schematic)
At the start: 20 parts, among them Q1 PMOS, Q3 PMOS, Q6 NMOS, Q7 NMOS, U11 MM3220AA2NRH

Commit message: Hardware revision 0.2 routing
Parts:
- BT3, BT4: footprint 254:BAT_254 -> Battery Holder - 18650:BAT_254
- Q6, Q7: value NMOS -> AOSP36326C
Connections:
- net 8.4unsafe: now reaches F5.1, Q3.1 (D)
- net d2d: now reaches Q6.1 (D), Q7.1 (D)
- net BATT- renamed BATT_LVL-
- net Cell1+ renamed BATT_LVL_MID
Other:
- company: (none) -> KBader94
- title: (none) -> OpenActionCam
Changed lines of the file:
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@@
 (kicad_sch (version 20230121) (generator eeschema)
   (paper "A4")
+  (title_block
+    (title "OpenActionCam")
+    (date "2025-04-10")
+    (rev "0.2")
+    (company "KBader94")
+    (comment 1 "https://github.com/kbader94/OpenActionCam")
+  )
   (junction (at 82.55 55.372) (diameter 0) (color 0 0 0 0)
   )
@@
   )
   (junction (at 226.822 43.688) (diameter 0) (color 0 0 0 0)
-  )
-  (junction (at 61.722 43.688) (diameter 0) (color 0 0 0 0)
   )
   (junction (at 104.394 119.634) (diameter 0) (color 0 0 0 0)
@@
     (stroke (width 0) (type default))
   )
-  (wire (pts (xy 35.814 43.688) (xy 61.722 43.688))
-    (stroke (width 0) (type default))
-  )
   (wire (pts (xy 168.148 84.074) (xy 202.692 84.074))
     (stroke (width 0) (type default))
@@
     (effects (font (size 1.27 1.27)) (justify left bottom))
   )
+  (label "8.4unsafe" (at 61.722 61.468 0) (fields_autoplaced)
+    (effects (font (size 1.27 1.27)) (justify left bottom))
+  )
   (label "Cell1+" (at 69.342 78.994 0) (fields_autoplaced)
     (effects (font (size 1.27 1.27)) (justify left bottom))
@@
     (effects (font (size 1.27 1.27)) (justify left bottom))
   )
-  (label "BATT+" (at 39.624 43.688 0) (fields_autoplaced)
-    (effects (font (size 1.27 1.27)) (justify left bottom))
-  )
-  (label "BATT+" (at 87.122 43.688 0) (fields_autoplaced)
+  (label "d2d" (at 197.612 119.634 0) (fields_autoplaced)
     (effects (font (size 1.27 1.27)) (justify left bottom))
   )
@@
     )
   )
-  (global_label "BATT-" (shape input) (at 40.894 119.634 180) (fields_autoplaced)
+  (global_label "BATT_LVL-" (shape input) (at 40.894 119.634 180) (fields_autoplaced)
     (effects (font (size 1.27 1.27)) (justify right))
-    (property "Intersheetrefs" "${INTERSHEET_REFS}" (at 31.9475 119.634 0)
+    (property "Intersheetrefs" "${INTERSHEET_REFS}" (at 27.8351 119.634 0)
       (effects (font (size 1.27 1.27)) (justify right) hide)
     )
   )
-  (global_label "BATT+" (shape input) (at 35.814 43.688 180) (fields_autoplaced)
+  (global_label "BATT_LVL_MID" (shape input) (at 38.354 78.994 180) (fields_autoplaced)
     (effects (font (size 1.27 1.27)) (justify right))
-    (property "Intersheetrefs" "${INTERSHEET_REFS}" (at 26.8675 43.688 0)
-      (effects (font (size 1.27 1.27)) (justify right) hide)
-    )
-  )
-  (global_label "Cell1+" (shape input) (at 38.354 78.994 180) (fields_autoplaced)
-    (effects (font (size 1.27 1.27)) (justify right))
-    (property "Intersheetrefs" "${INTERSHEET_REFS}" (at 28.8028 78.994 0)
+    (property "Intersheetrefs" "${INTERSHEET_REFS}" (at 22.5737 78.994 0)
       (effects (font (size 1.27 1.27)) (justify right) hide)
     )
@@
     (pin "2")
     (instances
-      (project "iJet"
+      (project "OAC"
         (path "/e63e39d7-6ac0-4ffd-8aa3-1841a4541b55/800e290e-8cfb-4946-9373-3e863e65a993/958a8f8b-4f02-4f0b-8738-caa770ee5158"
           (reference "C27") (unit 1)
@@
     (pin "2")
     (instances
-      (project "iJet"
+      (project "OAC"
         (path "/e63e39d7-6ac0-4ffd-8aa3-1841a4541b55/800e290e-8cfb-4946-9373-3e863e65a993/958a8f8b-4f02-4f0b-8738-caa770ee5158"
           (reference "R32") (unit 1)
@@
     (pin "1")
     (instances
-      (project "iJet"
+      (project "OAC"
         (path "/e63e39d7-6ac0-4ffd-8aa3-1841a4541b55/800e290e-8cfb-4946-9373-3e863e65a993/958a8f8b-4f02-4f0b-8738-caa770ee5158"
           (reference "F5") (unit 1)
@@
       (effects (font (size 1.27 1.27)) (justify left))
     )
-    (property "Footprint" "254:BAT_254" (at 61.722 74.676 90)
+    (property "Footprint" "Battery Holder - 18650:BAT_254" (at 61.722 74.676 90)
       (effects (font (size 1.27 1.27)) hide)
     )
@@
     (pin "2")
     (instances
-      (project "iJet"
+      (project "OAC"
         (path "/e63e39d7-6ac0-4ffd-8aa3-1841a4541b55/800e290e-8cfb-4946-9373-3e863e65a993/958a8f8b-4f02-4f0b-8738-caa770ee5158"
           (reference "BT3") (unit 1)
@@
     (pin "2")
     (instances
-      (project "iJet"
+      (project "OAC"
         (path "/e63e39d7-6ac0-4ffd-8aa3-1841a4541b55/800e290e-8cfb-4946-9373-3e863e65a993/958a8f8b-4f02-4f0b-8738-caa770ee5158"
           (reference "R28") (unit 1)
@@
     (pin "3")
     (instances
-      (project "iJet"
+      (project "OAC"
         (path "/e63e39d7-6ac0-4ffd-8aa3-1841a4541b55/800e290e-8cfb-4946-9373-3e863e65a993/958a8f8b-4f02-4f0b-8738-caa770ee5158"
           (reference "Q1") (unit 1)
@@
     (pin "1")
     (instances
-      (project "iJet"
+      (project "OAC"
         (path "/e63e39d7-6ac0-4ffd-8aa3-1841a4541b55/800e290e-8cfb-4946-9373-3e863e65a993/958a8f8b-4f02-4f0b-8738-caa770ee5158"
           (reference "F4") (unit 1)
@@
       (effects (font (size 1.27 1.27)) (justify left))
     )
-    (property "Footprint" "254:BAT_254" (at 61.722 115.57 90)
+    (property "Footprint" "Battery Holder - 18650:BAT_254" (at 61.722 115.57 90)
       (effects (font (size 1.27 1.27)) hide)
     )
@@
     (pin "2")
     (instances
-      (project "iJet"
+      (project "OAC"
         (path "/e63e39d7-6ac0-4ffd-8aa3-1841a4541b55/800e290e-8cfb-4946-9373-3e863e65a993/958a8f8b-4f02-4f0b-8738-caa770ee5158"
           (reference "BT4") (unit 1)
@@
     (pin "3")
     (instances
-      (project "iJet"
+      (project "OAC"
         (path "/e63e39d7-6ac0-4ffd-8aa3-1841a4541b55/800e290e-8cfb-4946-9373-3e863e65a993/958a8f8b-4f02-4f0b-8738-caa770ee5158"
           (reference "Q3") (unit 1)
@@
     (pin "2")
     (instances
-      (project "iJet"
+      (project "OAC"
         (path "/e63e39d7-6ac0-4ffd-8aa3-1841a4541b55/800e290e-8cfb-4946-9373-3e863e65a993/958a8f8b-4f02-4f0b-8738-caa770ee5158"
           (reference "R29") (unit 1)
@@
     (pin "1")
     (instances
-      (project "iJet"
+      (project "OAC"
         (path "/e63e39d7-6ac0-4ffd-8aa3-1841a4541b55/800e290e-8cfb-4946-9373-3e863e65a993/958a8f8b-4f02-4f0b-8738-caa770ee5158"
           (reference "D13") (unit 1)
@@
     (pin "2")
     (instances
-      (project "iJet"
+      (project "OAC"
         (path "/e63e39d7-6ac0-4ffd-8aa3-1841a4541b55/800e290e-8cfb-4946-9373-3e863e65a993/958a8f8b-4f02-4f0b-8738-caa770ee5158"
           (reference "C29") (unit 1)
@@
   (symbol (lib_id "Simulation_SPICE:NMOS") (at 212.852 122.174 90) (unit 1)
     (in_bom yes) (on_board yes) (dnp no) (fields_autoplaced)
-    (property "Reference" "Q6" (at 212.852 112.522 90)
-      (effects (font (size 1.27 1.27)))
-    )
-    (property "Value" "NMOS" (at 212.852 115.062 90)
+    (property "Reference" "Q6" (at 212.852 113.03 90)
+      (effects (font (size 1.27 1.27)))
+    )
+    (property "Value" "AOSP36326C" (at 212.852 115.57 90)
       (effects (font (size 1.27 1.27)))
     )
@@
     (pin "2")
     (instances
-      (project "iJet"
+      (project "OAC"
         (path "/e63e39d7-6ac0-4ffd-8aa3-1841a4541b55/800e290e-8cfb-4946-9373-3e863e65a993/958a8f8b-4f02-4f0b-8738-caa770ee5158"
           (reference "Q6") (unit 1)
@@
     (pin "1")
     (instances
-      (project "iJet"
+      (project "OAC"
         (path "/e63e39d7-6ac0-4ffd-8aa3-1841a4541b55/800e290e-8cfb-4946-9373-3e863e65a993/958a8f8b-4f02-4f0b-8738-caa770ee5158"
           (reference "#PWR043") (unit 1)
@@
     (pin "2")
     (instances
-      (project "iJet"
+      (project "OAC"
         (path "/e63e39d7-6ac0-4ffd-8aa3-1841a4541b55/800e290e-8cfb-4946-9373-3e863e65a993/958a8f8b-4f02-4f0b-8738-caa770ee5158"
           (reference "C28") (unit 1)
@@
     (pin "5")
     (instances
-      (project "iJet"
+      (project "OAC"
         (path "/e63e39d7-6ac0-4ffd-8aa3-1841a4541b55/800e290e-8cfb-4946-9373-3e863e65a993/958a8f8b-4f02-4f0b-8738-caa770ee5158"
           (reference "U11") (unit 1)
@@
     (pin "1")
     (instances
-      (project "iJet"
+      (project "OAC"
         (path "/e63e39d7-6ac0-4ffd-8aa3-1841a4541b55/800e290e-8cfb-4946-9373-3e863e65a993/958a8f8b-4f02-4f0b-8738-caa770ee5158"
           (reference "C26") (unit 1)
@@
     (pin "1")
     (instances
-      (project "iJet"
+      (project "OAC"
         (path "/e63e39d7-6ac0-4ffd-8aa3-1841a4541b55/800e290e-8cfb-4946-9373-3e863e65a993/958a8f8b-4f02-4f0b-8738-caa770ee5158"
           (reference "D15") (unit 1)
@@
     (pin "2")
     (instances
-      (project "iJet"
+      (project "OAC"
         (path "/e63e39d7-6ac0-4ffd-8aa3-1841a4541b55/800e290e-8cfb-4946-9373-3e863e65a993/958a8f8b-4f02-4f0b-8738-caa770ee5158"
           (reference "R31") (unit 1)
@@
       (effects (font (size 1.27 1.27)))
     )
-    (property "Value" "NMOS" (at 191.008 126.238 90)
+    (property "Value" "AOSP36326C" (at 191.008 126.238 90)
       (effects (font (size 1.27 1.27)))
     )
@@
     (pin "2")
     (instances
-      (project "iJet"
+      (project "OAC"
         (path "/e63e39d7-6ac0-4ffd-8aa3-1841a4541b55/800e290e-8cfb-4946-9373-3e863e65a993/958a8f8b-4f02-4f0b-8738-caa770ee5158"
           (reference "Q7") (unit 1)
@@
     (pin "2")
     (instances
-      (project "iJet"
+      (project "OAC"
         (path "/e63e39d7-6ac0-4ffd-8aa3-1841a4541b55/800e290e-8cfb-4946-9373-3e863e65a993/958a8f8b-4f02-4f0b-8738-caa770ee5158"
           (reference "R33") (unit 1)
