File: hardware/LED_Driver/LED_Array.kicad_sch (KiCad schematic)
At the start: 44 parts, among them J10 Conn_01x02_Pin, J11 Conn_01x02_Pin, J12 Conn_01x02_Pin, J13 Conn_01x02_Pin, J14 Conn_01x02_Pin, J15 LED_Board_Header, J5 Conn_01x02_Pin, J6 Conn_01x03, J8 Conn_01x02_Pin, J9 Conn_01x02_Pin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

Commit message: Hardware cleanup & enclosure prototype
* Seperates the kicad project into seperate projects per PCB
* initial FreeCAD Assets and prototypes added
Parts:
- removed C12: 0.1uF, Capacitor_SMD:C_0603_1608Metric_Pad1.08x0.95mm_HandSolder, symbol Device:C
- removed D1, D3, D5, D7: 3W LED, LEDS - BEAD 3W LED:BEAD-3W-W-120-04, symbol Device:LED
- removed D9: WS2812B, LED_SMD:LED_WS2812B_PLCC4_5.0x5.0mm_P3.2mm, symbol LED:WS2812B
- removed J11, J12, J13, J14: Conn_01x02_Pin, Connector_PinHeader_2.54mm:PinHeader_1x02_P2.54mm_Vertical, symbol Connector:Conn_01x02_Pin
- removed J15: LED_Board_Header, Connector_PinHeader_2.54mm:PinHeader_1x03_P2.54mm_Vertical, symbol Connector_Generic:Conn_01x03
- removed R12: 0, Resistor_SMD:R_0603_1608Metric_Pad0.98x0.95mm_HandSolder, symbol Device:R
Connections:
- no-connect marks 1 -> 0
