File: hardware/LED_Driver/LED_Driver.kicad_pcb (KiCad board)
At the start: 2 copper layers, 103.3 x 39.9 mm, 126 parts, among them J1 GPIO, J10 Conn_01x02_Pin, J11 Conn_01x02_Pin, J12 Conn_01x02_Pin, J13 Conn_01x02_Pin, J14 Conn_01x02_Pin, J15 LED_Board_Header, J2 Conn_02x11_Counter_Clockwise, J3 ICSP Header, J4 Conn_01x11, J5 Conn_01x02_Pin, J6 Conn_01x03, J7 UART DEBUG, J8 Conn_01x02_Pin, J9 Conn_01x02_Pin, Q1 PMOS, Q2 NMOS, Q3 PMOS, Q6 AOSP36326C, Q7 AOSP36326C, SW1 Button - User Interface, SW2 Button - Reset, U1 CAT24C256, U11 MM3220AA2NRH, U2 LM2596S-ADJ, U3 MCP73213-A6SI_MF, U4 ATmega328-P, U5 PT4115, U6 PT4115, U7 PT4115, U8 PT4115, Y2 16 Mhz

Commit message: Hardware cleanup & enclosure prototype
* Seperates the kicad project into seperate projects per PCB
* initial FreeCAD Assets and prototypes added
Parts:
- removed BT3, BT4: Battery_Cell, Battery Holder - 18650:BAT_254
- removed C1: 100n, Capacitor_SMD:C_0603_1608Metric_Pad1.08x0.95mm_HandSolder
- removed C10: 330uF 10V Elec, Capacitor_SMD:C_Elec_6.3x7.7
- removed C11: 0.1uF 25V, Capacitor_SMD:C_0603_1608Metric_Pad1.08x0.95mm_HandSolder
- removed C12, C26, C29, C6: 0.1uF, Capacitor_SMD:C_0603_1608Metric_Pad1.08x0.95mm_HandSolder
- removed C13, C14, C17: 100nF, Capacitor_SMD:C_0603_1608Metric_Pad1.08x0.95mm_HandSolder
- removed C15, C16: 22 pF, Capacitor_SMD:C_0603_1608Metric_Pad1.08x0.95mm_HandSolder
- removed C19: 0.1uF 0603, Capacitor_SMD:C_0603_1608Metric_Pad1.08x0.95mm_HandSolder
- removed C20, C21: 10uF 0805, Capacitor_SMD:C_0603_1608Metric_Pad1.08x0.95mm_HandSolder
- removed C27: 0.1 uF, Capacitor_SMD:C_0603_1608Metric_Pad1.08x0.95mm_HandSolder
- removed C28: 0.1uF OPT, Capacitor_SMD:C_0603_1608Metric_Pad1.08x0.95mm_HandSolder
- removed C32, C33: 47uF, Resistor_SMD:R_1210_3225Metric_Pad1.30x2.65mm_HandSolder
- removed C34: 47uF - 1210, Resistor_SMD:R_1210_3225Metric_Pad1.30x2.65mm_HandSolder
- removed C5: 47uF 1210, Resistor_SMD:R_1210_3225Metric_Pad1.30x2.65mm_HandSolder
- removed C7: 47uF 1210, Capacitor_SMD:C_1210_3225Metric_Pad1.33x2.70mm_HandSolder
- removed C8: 100uF 16V, Capacitor_SMD:CP_Elec_6.3x7.7
- removed C9: 330uF Tant 2312, C _Tantalum - TAJC337K006RNJ:CAPPM6032X280N
- removed D1, D3, D5, D7: 3W LED, LEDS - BEAD 3W LED:BEAD-3W-W-120-04
- removed D10, D9: WS2812B, LED_SMD:LED_WS2812B_PLCC4_5.0x5.0mm_P3.2mm
- removed D11: 5.1V Zener, Diode_SMD:D_MiniMELF_Handsoldering
- removed D12: SS34, Diode_SMD:D_SMA_Handsoldering
- removed D13, D15: 9.1V Zener, Diode_SMD:D_MiniMELF_Handsoldering
- removed D14: SS24, Diode_SMD:D_SMA_Handsoldering
- removed D16: SMAJ11A, Diode_SMD:D_SMA_Handsoldering
- removed F1: 6A Polyfuse 2920, Fuse:Fuse_2920_7451Metric_Pad2.10x5.45mm_HandSolder
- removed F2: 2.2A Polyfuse 1210, Fuse:Fuse_1210_3225Metric_Pad1.42x2.65mm_HandSolder
- removed F3: 2.2A Polyfuse, Fuse:Fuse_1210_3225Metric_Pad1.42x2.65mm_HandSolder
- removed F4, F5: Polyfuse 6A 2920, Fuse:Fuse_2920_7451Metric_Pad2.10x5.45mm_HandSolder
- removed G***: LOGO, LOGO
- removed J1: GPIO, Module:Raspberry_Pi_Zero_Socketed_THT_FaceDown_MountingHoles
- removed J11, J12, J13, J14: Conn_01x02_Pin, Connector_PinHeader_2.54mm:PinHeader_1x02_P2.54mm_Vertical
- removed J15: LED_Board_Header, Connector_PinHeader_2.54mm:PinHeader_1x03_P2.54mm_Vertical
- removed J2: Conn_02x11_Counter_Clockwise, Board:Board_outline
- removed J3: ICSP Header, Connector_PinSocket_2.54mm:PinSocket_2x03_P2.54mm_Vertical
- removed J4: Conn_01x11, Board:Board_outline
- removed J7: UART DEBUG, Connector_PinSocket_2.54mm:PinSocket_2x02_P2.54mm_Vertical
- removed JP1: ID_WP, Jumper:SolderJumper-2_P1.3mm_Open_Pad1.0x1.5mm
- removed L5: 33uH, Inductor - 125CDMCCDS 33uH:IND_125CDMCCDS-330MC
- removed Q1, Q3: PMOS, FET - SI4435FDY:SO-8_VIS
- removed Q2: NMOS, FET - AOSP36326C:SOIC127P490X600X175-8N
- removed Q6, Q7: AOSP36326C, FET - AOSP36326C:SOIC127P490X600X175-8N
- removed R1, R2: 3.9k, Resistor_SMD:R_0603_1608Metric_Pad0.98x0.95mm_HandSolder
- removed R10: 1K 0603, Resistor_SMD:R_0603_1608Metric_Pad0.98x0.95mm_HandSolder
- removed R12: 0, Resistor_SMD:R_0603_1608Metric_Pad0.98x0.95mm_HandSolder
- removed R17, R20: 3.3K, Resistor_SMD:R_0603_1608Metric_Pad0.98x0.95mm_HandSolder
- removed R18, R19: 2K, Resistor_SMD:R_0603_1608Metric_Pad0.98x0.95mm_HandSolder
- removed R21, R23, R24, R7: 10K, Resistor_SMD:R_0603_1608Metric_Pad0.98x0.95mm_HandSolder
- removed R22: 15K, Resistor_SMD:R_0603_1608Metric_Pad0.98x0.95mm_HandSolder
- removed R25, R26: 10K, Resistor_SMD:R_0603_1608Metric
- removed R27: 1K 0603, Resistor_SMD:R_0603_1608Metric
- removed R28, R29: 100K, Resistor_SMD:R_0603_1608Metric
- removed R31, R32: 330, Resistor_SMD:R_0603_1608Metric
- removed R33: 2.2K, Resistor_SMD:R_0603_1608Metric
- removed R8: 220, Resistor_SMD:R_0603_1608Metric_Pad0.98x0.95mm_HandSolder
- removed R9: 3.1K 0603, Resistor_SMD:R_0603_1608Metric_Pad0.98x0.95mm_HandSolder
- removed the REF** at (236.3, 96.0)
- removed SW1: Button - User Interface, Button - PTS815 Tactile SW:SW4_PTS815 SJM 250 SMTR LFS_CNK
- removed SW2: Button - Reset, Button - PTS815 Tactile SW:SW4_PTS815 SJM 250 SMTR LFS_CNK
- removed U1: CAT24C256, CAT24C256WI-GT3:SOIC127P600X175-8N
- removed U11: MM3220AA2NRH, MM3220AA2NRH:IC_MM3220AA2NRH
- removed U2: LM2596S-ADJ, Package_TO_SOT_SMD:TO-263-5_TabPin3
- removed U3: MCP73213-A6SI_MF, MCP73213-A6SI_MF:SON50P300X300X100-11N
- removed U4: ATmega328-P, ATMEGA328-AU:QFP80P900X900X120-32N
- removed Y2: 16 Mhz, Crystal - 16MHz ECS_160_20_5PX_TR:XTAL_ECS-160-20-5PX-TR
Routing:
- net +5V: track 261.3 -> 0.00 mm, vias 4 -> 0
- net BATT_LVL_MID: track 153.6 -> 0.00 mm, vias 16 -> 0
- net GND: track 229.9 -> 126.7 mm, vias 6 -> 0
- net BATT_LVL-: track 103.0 -> 0.00 mm, vias 13 -> 0
- net /Power State/Reset: track 89.5 -> 0.00 mm, vias 3 -> 0
- net 8.4V: track 266.7 -> 178.0 mm, vias 13 -> 11
- net STAT_LED: track 81.3 -> 0.00 mm, vias 1 -> 0
- net Chrg_Stat: track 78.7 -> 0.00 mm, vias 1 -> 0
- net /Power BMS/8.4V Out: track 77.6 -> 0.00 mm, vias 6 -> 0
- net Button: track 66.3 -> 0.00 mm
- net Rx: track 61.5 -> 0.00 mm, vias 2 -> 0
- net /Power State/Pi_En: track 50.4 -> 0.00 mm, vias 2 -> 0
- net /GPIO24: track 46.1 -> 0.00 mm, vias 1 -> 0
- net Tx: track 45.9 -> 0.00 mm, vias 2 -> 0
- net Net-(D10-DIN): track 44.3 -> 0.00 mm, vias 2 -> 0
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- removed copper zone on F.Cu, net +12V
- removed copper zone on F.Cu, net +5V
- removed copper zone on B.Cu, net /Power BMS/8.4V Out
- removed copper zone on F.Cu, net /Power BMS/8.4V Out
- removed copper zone on F.Cu, net /Power BMS/Battery Pack & Protection/8.4unsafe
- removed copper zone on F.Cu, net /Power BMS/Battery Pack & Protection/d2d
- removed copper zone on F.Cu, net /Power BMS/Power Supply/V_Out_Dirty
- removed copper zone on F.Cu, net /Power BMS/Power Supply/Vin_clean
- removed copper zone on F.Cu, net 8.4V
- removed copper zone on F.Cu, net BATT_LVL-
- removed copper zone on F.Cu, net BATT_LVL_MID
- removed copper zone on F.Cu, net GND
- removed copper zone on B.Cu, net Pi_Gnd
- removed copper zone on F.Cu, net Pi_Gnd
Other:
- board size 103.3 x 39.9 mm -> 39.9 x 39.9 mm
- board text removed: "ICSP"
- board text removed: "OpenActionCam"
- board text removed: "Power / Record"
- board text removed: "Reset"
- board text removed: "UART 5V"
- board text removed: "V 0.2 - 2025 - KBader94 https://github.com/kbader94/OpenActionCam"
