File: hardware/BMS/BMS.kicad_pcb (KiCad board)
At the start: 2 copper layers, 103.3 x 39.9 mm, 44 parts, among them J4 Conn_01x11, Q1 PMOS, Q3 PMOS, Q6 AOSP36326C, Q7 AOSP36326C, U11 MM3220AA2NRH, U2 LM2596S-ADJ, U3 MCP73213-A6SI_MF

Commit message: Hardware - Controller - Rev 0.3
* Consolidate various asset dirs into single symlinked directory.
* Fixes major flaw with previous atmega328 layout - wrong schematic symbol caused incorrect routing
* Use smaller crystal closer to mcu
* Add QR to silkscreen
Parts:
- C10: value 330uF 10V Elec -> 330uF 10V
- C11: renamed from C19; value 0.1uF 0603 -> 0.1uF
- C14: renamed from C28; value 0.1uF OPT -> 0.1uF
- C20, C21: value 10uF 0805 -> 10uF
- C34: value 47uF - 1210 -> 47uF
- C6: renamed from C5; value 47uF 1210 -> 47uF
- C8: renamed from C11; value 0.1uF 25V -> 0.1uF
- C9: value 330uF Tant 2312 -> 330uF Tantalum
- F1: renamed from F2; value 2.2A Polyfuse 1210 -> 2.2A Polyfuse
- F2: renamed from F1; value 6A Polyfuse 2920 -> 6A Polyfuse
- F4: renamed from F5; value Polyfuse 6A 2920 -> Polyfuse 6A
- F5: renamed from F4; value Polyfuse 6A 2920 -> Polyfuse 6A
- Q1: renamed from Q3; value PMOS -> SI4435FDY
- Q2: renamed from Q1; value PMOS -> SI4435FDY
- R2: renamed from R10; value 1K 0603 -> 1K
- R27: value 1K 0603 -> 1K
- R3: renamed from R9; value 3.1K 0603 -> 3.1K
- renumbered C26 to C12, C27 to C13, C29 to C15, C33 to C4, C32 to C5, C8 to C7, D12 to D3, D13 to D4, D15 to D5, L5 to L1, Q7 to Q3, Q6 to Q4, R29 to R4, R28 to R5, R32 to R6, R31 to R7, R33 to R8, U3 to U1, U11 to U3
Routing:
- net Net-(BT3-+): track 25.3 -> 23.9 mm
Other:
- board text added: "+12V IN"
- board text added: "+3.7V NOM OUT"
- board text added: "+5V OUT"
- board text added: "+7.4V NOM OUT"
- board text added: "CHRG STAT OUT"
- board text added: "GND"
