File: hardware/BMS/Power Boost.kicad_sch (KiCad schematic)
At the start: 10 parts, among them J4 Conn_01x11, U3 MCP73213-A6SI_MF

Commit message: Hardware - Controller - Rev 0.3
* Consolidate various asset dirs into single symlinked directory.
* Fixes major flaw with previous atmega328 layout - wrong schematic symbol caused incorrect routing
* Use smaller crystal closer to mcu
* Add QR to silkscreen
Parts:
- renumbered F1 to F2, U3 to U1
