File: hardware/Controller/Controller.kicad_sch (KiCad schematic)
At the start: 11 parts, among them J1 GPIO, J2 Conn_02x11_Counter_Clockwise, U1 CAT24C256

Commit message: Hardware - Controller - Rev 0.3
* Consolidate various asset dirs into single symlinked directory.
* Fixes major flaw with previous atmega328 layout - wrong schematic symbol caused incorrect routing
* Use smaller crystal closer to mcu
* Add QR to silkscreen
Parts:
- U1: footprint CAT24C256WI-GT3:SOIC127P600X175-8N -> IC - CAT24C256WI-GT3:SOIC127P600X175-8N
Changed lines of the file:
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@@
 			)
 		)
-		(property "Footprint" "CAT24C256WI-GT3:SOIC127P600X175-8N"
+		(property "Footprint" "IC - CAT24C256WI-GT3:SOIC127P600X175-8N"
 			(at 81.28 177.8 0)
 			(effects
